Commit message: no_ee

File: Rock-Walk/rock_walk/resources/models/end_effector.urdf (robot description, URDF)
Before this commit: robot EndEffector, 4 links, 3 joints
Links:
- link eef_link: geometry collision mesh filename=mesh/right_angle_eef_vhacd.obj; visual mesh filename=mesh/right_angle_eef.obj

File: Rock-Walk/rock_walk/resources/models/plane.urdf (robot description, URDF)
Before this commit: robot plane, 1 links, 0 joints
Links:
- link planeLink: geometry collision box size=100 100 10; visual mesh filename=mesh/plane.obj scale=1 1 1
