Commit message: object generation

File: Rock-Walk/rock_walk/resources/models/auto_object.urdf (robot description, URDF)
Before this commit: robot LargeConeControl, 5 links, 4 joints
Links:
- removed link apex_link_dummy
- added link apex_link_dummy_1, mass 0.0001
- added link apex_link_dummy_2, mass 0.0001
- added link cone, mass 1.922933964087465; collision mesh filename=mesh/object_mesh.obj; visual mesh filename=mesh/object_mesh.obj
Joints:
- removed joint joint_apex_dummy
- added joint joint_apex_dummy_1: type spherical, parent apex_link_z, child apex_link_dummy_1, axis 0 0 1
- added joint joint_apex_dummy_2: type spherical, parent apex_link_dummy_1, child apex_link_dummy_2, axis 0 1 0
- added joint joint_apex_dummy_3: type spherical, parent apex_link_dummy_2, child cone, axis 1 0 0

Commit message: update single_object_robust_quadrotor branch

File: Rock-Walk/rock_walk/resources/models/auto_object.urdf (robot description, URDF)
Before this commit: robot AutoObjectTransport, 7 links, 6 joints
Links:
- link cone: mass 1.6665427688758028 -> 1.8728423076371943
